File: PCB/RC Transmitter KiCad/RC Transmitter KiCad.kicad_pcb (KiCad board)
At the start: 2 copper layers, 15 parts, among them J1 J5019 Charger, J2 Conn_01x02_Socket, SW1 SW_DIP_x01, U2 HT7333-3.3_TO92, U3 Level Shifter TXS0108EPW

Commit message: updates
Parts:
- added C3: C 0.1u, Capacitor_THT:CP_Radial_D10.0mm_P5.00mm, F.Cu at (370.8, 157.5)
- added R1: R 10k, Resistor_THT:R_Axial_DIN0207_L6.3mm_D2.5mm_P5.08mm_Vertical, F.Cu at (331.1, 154.5)
- added R2: R 10k, Resistor_THT:R_Axial_DIN0207_L6.3mm_D2.5mm_P5.08mm_Vertical, F.Cu at (331.1, 158.6)
- added R3: R 10k, Resistor_THT:R_Axial_DIN0207_L6.3mm_D2.5mm_P5.08mm_Vertical, F.Cu at (331.1, 162.6)
- added R4: R 10k, Resistor_THT:R_Axial_DIN0207_L6.3mm_D2.5mm_P5.08mm_Vertical, F.Cu at (331.1, 166.7)
- added R5: R 10k, Resistor_THT:R_Axial_DIN0207_L6.3mm_D2.5mm_P5.08mm_Vertical, F.Cu at (331.1, 170.7)
- added R6: R 10k, Resistor_THT:R_Axial_DIN0207_L6.3mm_D2.5mm_P5.08mm_Vertical, F.Cu at (331.1, 174.8)
- added R7: R 10k, Resistor_THT:R_Axial_DIN0207_L6.3mm_D2.5mm_P5.08mm_Vertical, F.Cu at (331.1, 178.8)
- added R8: R 10k, Resistor_THT:R_Axial_DIN0207_L6.3mm_D2.5mm_P5.08mm_Vertical, F.Cu at (331.1, 185.4)
- added SW2: RotaryEncoder_Switch, Rotary_Encoder:RotaryEncoder_Alps_EC11E-Switch_Vertical_H20mm, F.Cu at (180.7, 111.8)
- added SW3: SW_Push_Dual UI Back Button, Button_Switch_THT:SW_PUSH_6mm, F.Cu at (97.6, 111.8)
- added SW4: SW_Push Left Bumper, Connector_PinHeader_2.00mm:PinHeader_1x02_P2.00mm_Vertical, F.Cu at (55.9, 43.2)
- added SW5: SW_Push Right Bumper, Connector_PinHeader_2.00mm:PinHeader_1x02_P2.00mm_Vertical, F.Cu at (243.8, 35.6)
- added U1: SN74HC165N, AddedFootprints:DIP794W45P254L1969H508Q16, F.Cu at (374.8, 247.7)
Connections:
- A1 pad 10: /TFT DC (D7) -> /TFT CS (D7)
- A1 pad 11: /Touch Screen CS (D8) -> /TFT DC (D8)
- A1 pad 12: /TFT Reset (D9) -> /Touch Screen CS (D9)
- A1 pad 13: unconnected-(A1-D10-Pad13) -> /TFT Reset (D10)
- A1 pad 5: /Joy Left Button (D2) -> /Shift Register Q7 (D2)
- A1 pad 6: /Joy Right Button (D3) -> /Shift Register PL (D3)
- A1 pad 7: /NRF CSN (D4) -> /Shift Register CP (D4)
- A1 pad 8: /NRF CE (D5) -> /NRF CSN (D5)
- A1 pad 9: /TFT CS (D6) -> /NRF CE (D6)
- N1 pad 2: /NRF CSN (D4) -> /NRF CSN (D5)
- N1 pad 7: /NRF CE (D5) -> /NRF CE (D6)
- U3 pad 13: /TFT Reset (D9) -> /TFT Reset (D10)
- U3 pad 14: /Touch Screen CS (D8) -> /Touch Screen CS (D9)
- U3 pad 15: /TFT DC (D7) -> /TFT DC (D8)
- U3 pad 16: /TFT CS (D6) -> /TFT CS (D7)

Commit message: progress
Parts:
- removed R1, R2, R3, R4, R5, R6, R7, R8: R 10k, Resistor_THT:R_Axial_DIN0207_L6.3mm_D2.5mm_P5.08mm_Vertical
- removed SW3: SW_Push_Dual UI Back Button, Button_Switch_THT:SW_PUSH_6mm
- added H1: MountingHole_Pad, MountingHole:MountingHole_2.2mm_M2, F.Cu at (85.1, 64.1)
- added H10: MountingHole_Pad, MountingHole:MountingHole_2.2mm_M2, F.Cu at (92.7, 110.5)
- added H2: MountingHole_Pad, MountingHole:MountingHole_2.2mm_M2, F.Cu at (215.9, 64.1)
- added H3: MountingHole_Pad, MountingHole:MountingHole_3.2mm_M3, F.Cu at (118.1, 134.6)
- added H4: MountingHole_Pad, MountingHole:MountingHole_3.2mm_M3, F.Cu at (178.4, 134.6)
- added H5: MountingHole_Pad, MountingHole:MountingHole_3.2mm_M3, F.Cu at (104.5, 68.6)
- added H6: MountingHole_Pad, MountingHole:MountingHole_3.2mm_M3, F.Cu at (196.5, 68.6)
- added H7: MountingHole_Pad, MountingHole:MountingHole_3.2mm_M3, F.Cu at (104.5, 118.1)
- added H8: MountingHole_Pad, MountingHole:MountingHole_3.2mm_M3, F.Cu at (196.5, 118.1)
- added H9: MountingHole_Pad, MountingHole:MountingHole_2.2mm_M2, F.Cu at (208.3, 110.5)
- added R10k_1: R 10k, Resistor_THT:R_Axial_DIN0207_L6.3mm_D2.5mm_P7.62mm_Horizontal, B.Cu at (182.9, 125.7)
- added R10k_2: R 10k, Resistor_THT:R_Axial_DIN0207_L6.3mm_D2.5mm_P7.62mm_Horizontal, B.Cu at (182.9, 120.0)
- added R10k_3: R 10k, Resistor_THT:R_Axial_DIN0207_L6.3mm_D2.5mm_P7.62mm_Horizontal, B.Cu at (171.4, 112.4)
- added R10k_4: R 10k, Resistor_THT:R_Axial_DIN0207_L6.3mm_D2.5mm_P7.62mm_Horizontal, B.Cu at (108.6, 123.8)
- added R10k_5: R 10k, Resistor_THT:R_Axial_DIN0207_L6.3mm_D2.5mm_P7.62mm_Horizontal, B.Cu at (108.6, 127.0)
- added R10k_6: R 10k, Resistor_THT:R_Axial_DIN0207_L6.3mm_D2.5mm_P7.62mm_Horizontal, B.Cu at (182.9, 116.8)
- added R10k_7: R 10k, Resistor_THT:R_Axial_DIN0207_L6.3mm_D2.5mm_P7.62mm_Horizontal, B.Cu at (99.1, 119.4)
- added R10k_8: R 10k, Resistor_THT:R_Axial_DIN0207_L6.3mm_D2.5mm_P7.62mm_Horizontal, B.Cu at (182.9, 128.9)
- added Tact_Push_Button_1: SW_Push Back, Button_Switch_THT:SW_PUSH_6mm, F.Cu at (102.2, 130.8)
- 1.27mm_JST_Connector_1: renamed from J2; moved to B.Cu
- Arduino_Nano_V3: renamed from A1; moved to B.Cu
- C10uf_1: renamed from C1; footprint Capacitor_THT:CP_Radial_D10.0mm_P5.00mm -> Capacitor_THT:CP_Radial_D5.0mm_P2.50mm; moved to B.Cu
- C10uf_2: renamed from C3; value C 0.1u -> C 10uf; footprint Capacitor_THT:CP_Radial_D10.0mm_P5.00mm -> Capacitor_THT:CP_Radial_D5.0mm_P2.50mm; moved to B.Cu
- C10uf_3: renamed from C2; footprint Capacitor_THT:CP_Radial_D10.0mm_P5.00mm -> Capacitor_THT:CP_Radial_D5.0mm_P2.50mm; moved to B.Cu
- HT7333-A_1: renamed from U2; moved to B.Cu
- J5019_1: renamed from J1; moved to B.Cu
- MPU6050_1: renamed from G1; moved to B.Cu
- NRF24L01+PA+LNA1: renamed from N1; moved to B.Cu
- SN74HC165N1: renamed from U1; value SN74HC165N -> SN74HC165N Shift Register; moved to B.Cu
- SPST_6A_Mini_Toggle_Switch_1: renamed from SW1; footprint AddedFootprints:SPST Mini Toggle Switch 2 Pin 2 Position -> Connector_PinHeader_2.00mm:PinHeader_1x02_P2.00mm_Vertical
- TXS0108E_1: renamed from U3; moved to B.Cu
- ‎PTV09A_1: renamed from RV2; footprint Potentiometer_THT:Potentiometer_ACP_CA9-V10_Vertical -> Potentiometer_THT:Potentiometer_Bourns_PTV09A-1_Single_Vertical
- ‎PTV09A_2: renamed from RV1; footprint Potentiometer_THT:Potentiometer_ACP_CA9-V10_Vertical -> Potentiometer_THT:Potentiometer_Bourns_PTV09A-1_Single_Vertical
- moved SN74HC165N1 277.0 mm to (127.6, 122.6)
- moved C10uf_2 235.8 mm to (136.5, 131.4), turned to 90 degrees
- moved HT7333-A_1 229.5 mm to (188.6, 106.7), turned to 180 degrees
- moved C10uf_3 214.1 mm to (188.6, 113.7), turned to 180 degrees
- moved C10uf_1 185.3 mm to (196.2, 106.7)
- moved 1.27mm_JST_Connector_1 171.3 mm to (111.1, 115.6), turned to 180 degrees
- moved NRF24L01+PA+LNA1 155.8 mm to (194.9, 98.4), turned to 90 degrees
- moved MPU6050_1 150.3 mm to (157.5, 90.8), turned to 180 degrees
- moved TXS0108E_1 127.5 mm to (109.9, 107.3)
- moved Arduino_Nano_V3 120.3 mm to (163.8, 102.2)
- moved J5019_1 92.7 mm to (172.3, 136.5), turned to 90 degrees
- moved SPST_6A_Mini_Toggle_Switch_1 59.2 mm to (85.1, 80.0)
- moved KW12_2 44.0 mm to (209.8, 63.5), turned to 90 degrees
- moved THB001P_2 42.0 mm to (210.6, 86.2)
- moved KW12_1 41.0 mm to (91.4, 63.5), turned to -90 degrees
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- renumbered SW2 to EC11E_1, S2 to ILI9488_1, SW4 to KW12_1, SW5 to KW12_2, JLeft1 to THB001P_1, JRight1 to THB001P_2
Connections:
- Arduino_Nano_V3 pad 17: unconnected-(A1-3V3-Pad17) -> /3.3v
- Arduino_Nano_V3 pad 19: /Joy Left X (A0) -> /Joy Left Y (A0)
- Arduino_Nano_V3 pad 20: /Joy Left Y (A1) -> /Joy Left X (A1)
- Arduino_Nano_V3 pad 21: /Joy Right X (A2) -> /Pot Left (A6)
- Arduino_Nano_V3 pad 22: /Joy Right Y (A3) -> /Joy Right X (A2)
- Arduino_Nano_V3 pad 25: /Pot Left (A6) -> /Joy Right Y (A3)
- C10uf_1 pad 1: /3.3v -> Net-(HT7333-A_1-VO)
- C10uf_3 pad 1: /3.3v -> Net-(HT7333-A_1-VO)
- HT7333-A_1 pad 1: /3.3v -> Net-(HT7333-A_1-VO)
- NRF24L01+PA+LNA1 pad 1: /3.3v -> Net-(HT7333-A_1-VO)
- SN74HC165N1 pad 14: /Joy Left Button (D2) -> /Joy Right Button (D3)
- SN74HC165N1 pad 3: /Joy Right Button (D3) -> /Joy Left Button (D2)
- THB001P_1 pad 12: /Joy Left Y (A1) -> /Joy Left Y (A0)
- THB001P_1 pad 2: /Joy Left X (A0) -> /Joy Left X (A1)
Routing:
- net /5v: track 0.00 -> 468.2 mm, vias 0 -> 4
- net /Pot Right (A7): track 0.00 -> 183.1 mm
- net Net-(SN74HC165N1-D7): track 0.00 -> 142.2 mm
- net /MOSI (D11): track 0.00 -> 134.6 mm
- net /MISO (D12): track 0.00 -> 124.5 mm
- net /SCK (D13): track 0.00 -> 124.1 mm
- net /Joy Left X (A1): track 0.00 -> 109.1 mm
- net /3.3v: track 0.00 -> 106.8 mm
- net /Joy Left Y (A0): track 0.00 -> 106.3 mm
- net Net-(SN74HC165N1-D6): track 0.00 -> 103.8 mm
- net Net-(J5019_1-BAT+): track 0.00 -> 95.0 mm
- net /Joy Right Button (D3): track 0.00 -> 93.6 mm
- net Net-(SN74HC165N1-D0): track 0.00 -> 82.4 mm
- net /Shift Register PL (D3): track 0.00 -> 70.8 mm
- net /Shift Register CP (D4): track 0.00 -> 70.8 mm
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- added copper zone on B.Cu, net GND
- added copper zone on F.Cu, net GND
Other:
- board outline added: 135.9 x 76.8 mm

Commit message: finished footprint for now
Parts:
- moved SPST_6A_Mini_Toggle_Switch_1 2.54 mm to (85.1, 82.5)
Routing:
- net /5v: track 468.2 -> 516.4 mm
- net /Shift Register Q7 (D2): track 47.2 -> 62.3 mm
- net /Joy Left X (A1): track 109.1 -> 120.3 mm
- net /Joy Left Y (A0): track 106.3 -> 114.7 mm
- net Net-(SN74HC165N1-D6): track 103.8 -> 95.7 mm
- net /Shift Register PL (D3): track 70.8 -> 78.1 mm
- net /TFT CS (D7): track 49.1 -> 55.6 mm
- net /TFT DC (D8): track 49.1 -> 54.4 mm
- net /Shift Register CP (D4): track 70.8 -> 76.0 mm
- net /Joy Right Button (D3): track 93.6 -> 89.2 mm
- net /Touch Screen CS (D9): track 49.1 -> 53.3 mm
- net /TFT Reset (D10): track 55.3 -> 52.2 mm
- net Net-(SN74HC165N1-D1): track 68.1 -> 71.1 mm
- net /3.3v: track 106.8 -> 109.8 mm
- net Net-(J5019_1-BAT+): track 95.0 -> 97.5 mm
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