File: PCB/RC Transmitter KiCad/RC Transmitter KiCad.kicad_sch (KiCad schematic)
At the start: 15 parts, among them J1 J5019 Charger, SW1 SW_DIP_x01, U2 HT7333-3.3_TO92, U3 Level Shifter TXS0108EPW

Commit message: updates
Parts:
- removed BT1: Battery_Cell, Connector_JST:JST_GH_BM02B-GHS-TBT_1x02-1MP_P1.25mm_Vertical, symbol Device:Battery_Cell
- added C3: C 0.1u, Capacitor_THT:CP_Radial_D10.0mm_P5.00mm, symbol Device:C
- added J2: Conn_01x02_Socket, Connector_PinSocket_1.27mm:PinSocket_1x02_P1.27mm_Vertical, symbol Connector:Conn_01x02_Socket
- added R1, R2, R3, R4, R5, R6, R7, R8: R 10k, Resistor_THT:R_Axial_DIN0207_L6.3mm_D2.5mm_P5.08mm_Vertical, symbol Device:R
- added SW2: RotaryEncoder_Switch, Rotary_Encoder:RotaryEncoder_Alps_EC11E-Switch_Vertical_H20mm, symbol Device:RotaryEncoder_Switch
- added SW3: SW_Push_Dual UI Back Button, Button_Switch_THT:SW_PUSH_6mm, symbol Switch:SW_Push_Dual
- added SW4: SW_Push Left Bumper, Connector_PinHeader_2.00mm:PinHeader_1x02_P2.00mm_Vertical, symbol Switch:SW_Push
- added SW5: SW_Push Right Bumper, Connector_PinHeader_2.00mm:PinHeader_1x02_P2.00mm_Vertical, symbol Switch:SW_Push
- added U1: SN74HC165N, AddedFootprints:DIP794W45P254L1969H508Q16, symbol 74xx:74HC165
Connections:
- net 5v: now also C3.1, R2.1, R3.1, SW2.S2, SW3.1, SW4.1, SW5.1, U1.16 (VCC)
- net GND: now also C3.2, R1.2, R4.1, R5.1, R6.1, R7.1, R8.1, SW2.C, U1.10 (DS), U1.15 (~{CE}), U1.8 (GND)
- net Joy Left Button (D2): now also R8.2, U1.14 (D3); no longer A1.5 (D2)
- net Joy Right Button (D3): now also R7.2, U1.3 (D4); no longer A1.6 (D3)
- net at SW1.2: now also J2.1 (Pin_1)
- net at J1.6 (BAT-): now also J2.2 (Pin_2)
- net TFT Reset (D10): now reaches A1.13 (D10)
- net TFT Reset (D10): now also U3.13 (B7)
- net NRF CE (D5) renamed NRF CE (D6)
- net NRF CE (D6): now also A1.9 (D6); no longer A1.8 (D5)
- net NRF CSN (D4) renamed NRF CSN (D5)
- net NRF CSN (D5): now also A1.8 (D5); no longer A1.7 (D4)
- net TFT CS (D6) renamed TFT CS (D7)
- net TFT CS (D7): now also A1.10 (D7); no longer A1.9 (D6)
- net TFT DC (D7) renamed TFT DC (D8)
- net TFT DC (D8): now also A1.11 (D8); no longer A1.10 (D7)
- net TFT Reset (D9) renamed Touch Screen CS (D9)
- net Touch Screen CS (D9): now also U3.14 (B6); no longer U3.13 (B7)
- removed net Touch Screen CS (D8): A1.11 (D8), U3.14 (B6)
- new net: R5.2, SW4.2, U1.5 (D6)
- new net: R2.2, SW2.A, U1.13 (D2)
- new net: R3.2, SW2.B, U1.12 (D1)
- new net: R1.1, SW2.S1, U1.11 (D0)
- new net: R6.2, SW3.2, U1.4 (D5)
- new net: R4.2, SW5.2, U1.6 (D7)
- new net Shift Register CP (D4): A1.7 (D4), U1.2 (CP)
- new net Shift Register PL (D3): A1.6 (D3), U1.1 (~{PL})
- new net Shift Register Q7 (D2): A1.5 (D2), U1.9 (Q7)
Other:
- moved on the sheet: C2, S2, SW1, U3

Commit message: progress
Parts:
- removed SW3: SW_Push_Dual UI Back Button, Button_Switch_THT:SW_PUSH_6mm, symbol Switch:SW_Push_Dual
- added H1, H10, H2, H9: MountingHole_Pad, MountingHole:MountingHole_2.2mm_M2, symbol Mechanical:MountingHole
- added H3, H4, H5, H6, H7, H8: MountingHole_Pad, MountingHole:MountingHole_3.2mm_M3, symbol Mechanical:MountingHole
- added Tact_Push_Button_1: SW_Push Back, Button_Switch_THT:SW_PUSH_6mm, symbol Switch:SW_Push
- C10uf_1: renamed from C1; footprint Capacitor_THT:CP_Radial_D10.0mm_P5.00mm -> Capacitor_THT:CP_Radial_D5.0mm_P2.50mm
- C10uf_2: renamed from C3; value C 0.1u -> C 10uf; footprint Capacitor_THT:CP_Radial_D10.0mm_P5.00mm -> Capacitor_THT:CP_Radial_D5.0mm_P2.50mm
- C10uf_3: renamed from C2; footprint Capacitor_THT:CP_Radial_D10.0mm_P5.00mm -> Capacitor_THT:CP_Radial_D5.0mm_P2.50mm
- R10k_1: renamed from R2; footprint Resistor_THT:R_Axial_DIN0207_L6.3mm_D2.5mm_P5.08mm_Vertical -> Resistor_THT:R_Axial_DIN0207_L6.3mm_D2.5mm_P7.62mm_Horizontal
- R10k_2: renamed from R3; footprint Resistor_THT:R_Axial_DIN0207_L6.3mm_D2.5mm_P5.08mm_Vertical -> Resistor_THT:R_Axial_DIN0207_L6.3mm_D2.5mm_P7.62mm_Horizontal
- R10k_3: renamed from R4; footprint Resistor_THT:R_Axial_DIN0207_L6.3mm_D2.5mm_P5.08mm_Vertical -> Resistor_THT:R_Axial_DIN0207_L6.3mm_D2.5mm_P7.62mm_Horizontal
- R10k_4: renamed from R5; footprint Resistor_THT:R_Axial_DIN0207_L6.3mm_D2.5mm_P5.08mm_Vertical -> Resistor_THT:R_Axial_DIN0207_L6.3mm_D2.5mm_P7.62mm_Horizontal
- R10k_5: renamed from R6; footprint Resistor_THT:R_Axial_DIN0207_L6.3mm_D2.5mm_P5.08mm_Vertical -> Resistor_THT:R_Axial_DIN0207_L6.3mm_D2.5mm_P7.62mm_Horizontal
- R10k_6: renamed from R1; footprint Resistor_THT:R_Axial_DIN0207_L6.3mm_D2.5mm_P5.08mm_Vertical -> Resistor_THT:R_Axial_DIN0207_L6.3mm_D2.5mm_P7.62mm_Horizontal
- R10k_7: renamed from R7; footprint Resistor_THT:R_Axial_DIN0207_L6.3mm_D2.5mm_P5.08mm_Vertical -> Resistor_THT:R_Axial_DIN0207_L6.3mm_D2.5mm_P7.62mm_Horizontal
- R10k_8: renamed from R8; footprint Resistor_THT:R_Axial_DIN0207_L6.3mm_D2.5mm_P5.08mm_Vertical -> Resistor_THT:R_Axial_DIN0207_L6.3mm_D2.5mm_P7.62mm_Horizontal
- SN74HC165N1: renamed from U1; value SN74HC165N -> SN74HC165N Shift Register
- SPST_6A_Mini_Toggle_Switch_1: renamed from SW1; footprint AddedFootprints:SPST Mini Toggle Switch 2 Pin 2 Position -> Connector_PinHeader_2.00mm:PinHeader_1x02_P2.00mm_Vertical
- ‎PTV09A_1: renamed from RV2; footprint Potentiometer_THT:Potentiometer_ACP_CA9-V10_Vertical -> Potentiometer_THT:Potentiometer_Bourns_PTV09A-1_Single_Vertical
- ‎PTV09A_2: renamed from RV1; footprint Potentiometer_THT:Potentiometer_ACP_CA9-V10_Vertical -> Potentiometer_THT:Potentiometer_Bourns_PTV09A-1_Single_Vertical
- renumbered J2 to 1.27mm_JST_Connector_1, A1 to Arduino_Nano_V3, SW2 to EC11E_1, U2 to HT7333-A_1, S2 to ILI9488_1, J1 to J5019_1, SW4 to KW12_1, SW5 to KW12_2, G1 to MPU6050_1, N1 to NRF24L01+PA+LNA1, JLeft1 to THB001P_1, JRight1 to THB001P_2, U3 to TXS0108E_1
Connections:
- net 3.3v: now also Arduino_Nano_V3.17 (3V3); no longer C10uf_1.1, C10uf_3.1, HT7333-A_1.1 (VO), NRF24L01+PA+LNA1.1 (V+)
- net 5v: now also Tact_Push_Button_1.1
- net Joy Left Button (D2): now also R10k_7.2, SN74HC165N1.3 (D4); no longer R10k_8.2, SN74HC165N1.14 (D3)
- net Joy Right Button (D3): now also R10k_8.2, SN74HC165N1.14 (D3); no longer R10k_7.2, SN74HC165N1.3 (D4)
- net Joy Right X (A2): now also Arduino_Nano_V3.22 (A3); no longer Arduino_Nano_V3.21 (A2)
- net Joy Right Y (A3): now also Arduino_Nano_V3.25 (A6); no longer Arduino_Nano_V3.22 (A3)
- net Pot Left (A6): now also Arduino_Nano_V3.21 (A2); no longer Arduino_Nano_V3.25 (A6)
- net at R10k_5.2, SN74HC165N1.4 (D5): now also Tact_Push_Button_1.2
- net Joy Left X (A0) renamed Joy Left X (A1)
- net Joy Left X (A1): now also Arduino_Nano_V3.20 (A1); no longer Arduino_Nano_V3.19 (A0)
- net Joy Left Y (A1) renamed Joy Left Y (A0)
- net Joy Left Y (A0): now also Arduino_Nano_V3.19 (A0); no longer Arduino_Nano_V3.20 (A1)
- new net: C10uf_1.1, C10uf_3.1, HT7333-A_1.1 (VO), NRF24L01+PA+LNA1.1 (V+)
- no-connect marks 22 -> 21
Other:
- note added: "Buttons"
- moved on the sheet: C10uf_2, EC11E_1, KW12_1, KW12_2, R10k_1, R10k_2, R10k_3, R10k_4, R10k_5, R10k_6, R10k_7, R10k_8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

Commit message: finished footprint for now
Parts:
- ILI9488_1: value Screen ILI9341 -> Screen ILI9488
Other:
- note added: "NRF"
Changed lines of the file:
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@@
     (effects (font (size 2 2)) (justify left bottom))
   )
-  (text "Potentiometers" (at 100.33 58.42 0)
+  (text "NRF\n" (at 100.33 58.42 0)
     (effects (font (size 2 2)) (justify left bottom))
   )
@@
       (effects (font (size 1.27 1.27)) (justify left))
     )
-    (property "Value" "Screen ILI9341" (at 177.8 123.19 0)
-      (effects (font (size 1.27 1.27)))
-    )
+    (property "Value" "Screen ILI9488" (at 177.8 123.19 0)
+      (effects (font (size 1.27 1.27)))
+    )
