File: PCB/RCTransmitter/RCTransmitterAecertRobotics.kicad_sch (KiCad schematic)
At the start: 41 parts, among them K1 KCD1 Power Switch

Commit message: nrf stuff
Parts:
- removed Level_Shifter1: TXS0108EPW, AddedFootprints:HW-221 Level Shifter, symbol Logic_LevelTranslator:TXS0108EPW
- removed Touch_Screen1: Hosyond 3.5 Inch TFT Touch Screen ILI9488, AddedFootprints:3.5 Inch Screen SPI_Module_ILI9488, symbol Modules:2.8inch_SPI_Module_ILI9341
- added OLED_LCD_Display1: SSD1309 2.4inch, AddedFootprints:OLED LCD Display SSD1309, symbol Modules:SSD1309_2.4_Inch_OLED
- H1, H10, H2, H9: footprint MountingHole:MountingHole_2.2mm_M2 -> MountingHole:MountingHole_3.2mm_M3
Connections:
- net SCL (A5) is gone; now on net SCL: Gyroscope1.3 (SCL), IO_Extender1.22 (SCL)
- net SDA (A4) is gone; now on net SDA: Gyroscope1.4 (SDA), IO_Extender1.21 (SDA)
- net TFT Reset is gone; now on net Joy Left Button: IO_Extender1.0 (P00)
- net 5v: now also Bumper1.1, Bumper2.1, Bumper3.1, Bumper4.1, Button1.1, Button2.1, Button3.1, Button4.1, Toggle_Switch1.1, Toggle_Switch2.1, Toggle_Switch3.1, Toggle_Switch4.1, OLED_LCD_Display1.6 (VCC); no longer 3.3V_Regulator1.2 (VI), Battery_Charger1.1 (VOUT+), K1.1 (LED)
- net Button A: now also IO_Extender1.13 (P13); no longer IO_Extender1.1 (P01)
- net Button B: now also IO_Extender1.12 (P12); no longer IO_Extender1.2 (P02)
- net Button C: now also IO_Extender1.11 (P11); no longer IO_Extender1.3 (P03)
- net Button D: now also IO_Extender1.10 (P10); no longer IO_Extender1.4 (P04)
- net GND: now also K1.1 (LED), OLED_LCD_Display1.7 (GND); no longer Battery_Charger1.2 (VOUT-), Bumper1.1, Bumper2.1, Bumper3.1, Bumper4.1, Button1.1, Button2.1, Button3.1, Button4.1, Toggle_Switch1.1, Toggle_Switch2.1, Toggle_Switch3.1, Toggle_Switch4.1
- net Joy Left Button: no longer IO_Extender1.5 (P05)
- net Joy Left X: now also Arduino_Nano_V3.26 (A7); no longer Arduino_Nano_V3.21 (A2)
- net Joy Left Y: now also Arduino_Nano_V3.25 (A6); no longer Arduino_Nano_V3.20 (A1)
- net Joy Right Button: now also IO_Extender1.1 (P01); no longer IO_Extender1.17 (P17)
- net Joy Right X: now also Arduino_Nano_V3.21 (A2); no longer Arduino_Nano_V3.22 (A3)
- net Joy Right Y: now also Arduino_Nano_V3.22 (A3); no longer Arduino_Nano_V3.25 (A6)
- net Left Bumper A: now also IO_Extender1.14 (P14); no longer IO_Extender1.7 (P07)
- net Left Bumper B: now also IO_Extender1.17 (P17); no longer IO_Extender1.6 (P06)
- net MOSI: now also OLED_LCD_Display1.4 (SDA)
- net Pot Right: now also Arduino_Nano_V3.20 (A1); no longer Arduino_Nano_V3.26 (A7)
- net Right Bumper A: now also IO_Extender1.5 (P05); no longer IO_Extender1.14 (P14)
- net Right Bumper B: now also IO_Extender1.4 (P04); no longer IO_Extender1.13 (P13)
- net Rotary Encoder Switch: now also IO_Extender1.6 (P06); no longer IO_Extender1.12 (P12)
- net SCK: now also OLED_LCD_Display1.5 (SCK)
- net Toggle A: now also IO_Extender1.15 (P15); no longer IO_Extender1.10 (P10)
- net Toggle B: now also IO_Extender1.16 (P16); no longer IO_Extender1.11 (P11)
- net Toggle C: now also IO_Extender1.2 (P02); no longer IO_Extender1.16 (P16)
- net Toggle D: now also IO_Extender1.3 (P03); no longer IO_Extender1.15 (P15)
- net at K1.2 (Power): now also Battery_Charger1.2 (VOUT-); no longer Battery_Charger1.5 (BAT+)
- net at JST_Connector1.1 (Pin_1): now also Battery_Charger1.5 (BAT+); no longer K1.3 (Ground)
- net Vin: now reaches Arduino_Nano_V3.30 (VIN)
- net Vin: now also 3.3V_Regulator1.2 (VI), Battery_Charger1.1 (VOUT+), K1.3 (Load)
- net TFT CS renamed Screen RES
- net Screen RES: now also OLED_LCD_Display1.3 (RES)
- net TFT DC renamed Screen DC
- net Screen DC: now also OLED_LCD_Display1.2 (DC)
- net Touch Screen CS renamed Screen CS
- net Screen CS: now also OLED_LCD_Display1.1 (CS)
- no-connect marks 23 -> 14
Other:
- moved on the sheet: Battery_Charger1, H1, H2, H3, H4, H5, H6, H7, H8, JST_Connector1
