File: RC_V2/PCB Mega Mini/RCTransmitterAecertRobotics.kicad_sch (KiCad schematic)
At the start: 39 parts

Commit message: Neatened up schematic
Other:
- note added: "Buttons, Toggles, Bumpers"
- note added: "Power"
- note added: "Rotary Encoder"
- note removed: "Battery Stuff"
- note removed: "Buttons, Toggles, Bumpers, Rotary Encoder, and IO Extender"
- moved on the sheet: Arduino_Mega_Pro1, Bumper1, Bumper2, Bumper3, Bumper4, Button1, Button2, Button3, Button4, C1, C2, Gyroscope1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
